File: hs_wpi_test_board.sch (KiCad schematic (older format))
At the start: 34 parts, among them J1 Raspberry_Pi_2_3, Q1 Q_NPN_EBC, Q10 Q_NPN_EBC, Q2 Q_NPN_EBC, Q3 Q_NPN_EBC, Q4 Q_NPN_EBC, Q5 Q_NPN_EBC, Q6 Q_NPN_EBC, Q7 Q_NPN_EBC, Q8 Q_NPN_EBC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

Commit message: pin header straight
Parts:
- J1: footprint Socket_Strips:Socket_Strip_Angled_2x20_Pitch2.54mm -> Pin_Headers:Pin_Header_Straight_2x20_Pitch2.54mm
Changed lines of the file:
@@
 F 0 "J1" H 5850 4950 50  0000 C CNN
 F 1 "Raspberry_Pi_2_3" H 4750 7100 50  0000 C CNN
-F 2 "Socket_Strips:Socket_Strip_Angled_2x20_Pitch2.54mm" H 6150 7450 50  0001 C CNN
+F 2 "Pin_Headers:Pin_Header_Straight_2x20_Pitch2.54mm" H 6150 7450 50  0001 C CNN
 F 3 "" H 5200 6050 50  0001 C CNN
 	1    5150 6200

Commit message: angled socket
Parts:
- J1: footprint Pin_Headers:Pin_Header_Straight_2x20_Pitch2.54mm -> Socket_Strips:Socket_Strip_Angled_2x20_Pitch2.54mm
Changed lines of the file:
@@
 F 0 "J1" H 5850 4950 50  0000 C CNN
 F 1 "Raspberry_Pi_2_3" H 4750 7100 50  0000 C CNN
-F 2 "Pin_Headers:Pin_Header_Straight_2x20_Pitch2.54mm" H 6150 7450 50  0001 C CNN
+F 2 "Socket_Strips:Socket_Strip_Angled_2x20_Pitch2.54mm" H 6150 7450 50  0001 C CNN
 F 3 "" H 5200 6050 50  0001 C CNN
 	1    5150 6200
