File: hs_wpi_test_board.kicad_pcb (KiCad board)
At the start: 2 copper layers, 57.2 x 52.1 mm, 34 parts, among them J1 Raspberry_Pi_2_3, Q1 Q_NPN_EBC, Q10 Q_NPN_EBC, Q2 Q_NPN_EBC, Q3 Q_NPN_EBC, Q4 Q_NPN_EBC, Q5 Q_NPN_EBC, Q6 Q_NPN_EBC, Q7 Q_NPN_EBC, Q8 Q_NPN_EBC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

Commit message: finished board
Routing:
- net Net-(J1-Pad31): track 88.7 -> 60.1 mm
- net GND: track 0.00 -> 12.1 mm
- added copper zone on B.Cu, net GND
Changed lines of the file:
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@@
   (general
     (links 65)
-    (no_connects 20)
+    (no_connects 0)
     (area 104.781886 73.333789 162.635001 129.7024)
     (thickness 1.6)
     (drawings 4)
-    (tracks 246)
+    (tracks 251)
     (zones 0)
     (modules 34)
@@
   (gr_line (start 162.56 76.2) (end 162.56 128.27) (angle 90) (layer Edge.Cuts) (width 0.15))
   (gr_line (start 105.41 76.2) (end 162.56 76.2) (angle 90) (layer Edge.Cuts) (width 0.15))
+  (segment (start 122.555 81.28) (end 121.476399 80.201399) (width 0.1524) (layer F.Cu) (net 1))
+  (segment (start 121.476399 80.201399) (end 118.553601 80.201399) (width 0.1524) (layer F.Cu) (net 1))
+  (segment (start 118.553601 80.201399) (end 118.324999 80.430001) (width 0.1524) (layer F.Cu) (net 1))
+  (segment (start 118.324999 80.430001) (end 117.475 81.28) (width 0.1524) (layer F.Cu) (net 1))
+  (segment (start 127.635 78.74) (end 126.556399 79.818601) (width 0.1524) (layer F.Cu) (net 1))
+  (segment (start 126.556399 79.818601) (end 124.016399 79.818601) (width 0.1524) (layer F.Cu) (net 1))
+  (segment (start 124.016399 79.818601) (end 123.404999 80.430001) (width 0.1524) (layer F.Cu) (net 1))
+  (segment (start 123.404999 80.430001) (end 122.555 81.28) (width 0.1524) (layer F.Cu) (net 1))
   (segment (start 109.22 102.235) (end 109.22 107.315) (width 0.25) (layer F.Cu) (net 2))
   (segment (start 109.22 107.315) (end 110.49 108.585) (width 0.25) (layer F.Cu) (net 2))
@@
   (segment (start 121.802153 116.647401) (end 122.362401 116.087153) (width 0.25) (layer F.Cu) (net 34))
   (segment (start 120.767847 116.647401) (end 121.802153 116.647401) (width 0.25) (layer F.Cu) (net 34))
-  (segment (start 122.362401 111.729847) (end 118.11 107.477446) (width 0.25) (layer F.Cu) (net 34))
-  (segment (start 122.362401 116.087153) (end 122.362401 111.729847) (width 0.25) (layer F.Cu) (net 34))
-  (segment (start 118.11 107.477446) (end 118.11 125.73) (width 0.25) (layer F.Cu) (net 34))
   (segment (start 122.362401 116.087153) (end 122.362401 111.895818) (width 0.25) (layer F.Cu) (net 34))
   (segment (start 120.340188 109.873605) (end 120.340188 101.909812) (width 0.25) (layer F.Cu) (net 34))
@@
   (segment (start 139.5436 125.73) (end 132.57637 125.73) (width 0.25) (layer F.Cu) (net 36))
   (segment (start 132.57637 125.73) (end 131.445 125.73) (width 0.25) (layer F.Cu) (net 36))
+  (zone (net 1) (net_name GND) (layer B.Cu) (hatch edge 0.508)
+    (connect_pads (clearance 0.508))
+    (min_thickness 0.254)
+    (fill yes (arc_segments 16) (thermal_gap 0.508) (thermal_bridge_width 0.508))
+    (polygon
+      (pts
+        (xy 162.56 128.27) (xy 105.41 128.27) (xy 105.41 76.2) (xy 162.56 76.2)
+      )
+    )
+  )
 )

Commit message: switch J1 footprint to Connectors:IDC_Header_Straight_40pins
Parts:
- J1: footprint Pin_Headers:Pin_Header_Straight_2x20_Pitch2.54mm -> Connectors:IDC_Header_Straight_40pins
- turned J1 to 180 degrees
Routing:
- net Net-(J1-Pad29): track 61.8 -> 63.3 mm
